File: assets/watch_v1/watch_v1.kicad_sch (KiCad schematic)
At the start: 8 parts

Commit message: Design watch_v1 KiCad schematic and PCB in assets/
- Consolidated KiCad project into assets/watch_v1/ (canonical location)
- Fully wired schematic: ESP32-C3, 5643A-1 display, TP4056, Schottky, MCP1700-33 LDO,
  2N2222 digit drivers, buttons, LDR, RGB LED, vibration motor, resistors, caps
- PCB: 60x40mm outline, 40 footprints, 40 nets, 4 mounting holes, net classes
- Fixed LDO_OUT power-short bug (separated 3.3V rail from 5V VBUS)
- Removed temp files: .hermes-tmp.*, *.bak, fp-info-cache
- Removed duplicate KiCad files from src/
- .gitignore: ignore KiCad backup/cache artifacts
- Updated TODO.md, docs/README.md, docs/BUILD_GUIDE.md paths
Parts:
- removed ? (x8): (no value)
Other:
- title: ESP32-C3 SuperMini Watch -> (none)
