File: assets/watch_v1/watch_v1.kicad_sch (KiCad schematic)
At the start: 0 parts

Commit message: Fix schematic top-level S-expression structure
- Wrapped all elements inside single (kicad_sch ...) group (was separate top-level groups)
- KiCad 10.0 eeschema loads successfully
- 39 symbols, 91 wires, 44 labels — balanced S-expression
- LDO_OUT connected to 3V3 rail, U1.VBUS connected to VBUS rail
Parts:
- added BT1: 3.7V 150mAh Li-Po, Connector:JST_PH_2pin
- added C1, C2: 1uF, Capacitor_THT:CP_Radial_D5.0mm_P2.50mm
- added D1: 1N5819 Schottky (BAT→LDO), Package_TO_SOT_SMD:DO-41
- added D2: 1N5819 Schottky (USB→LDO), Package_TO_SOT_SMD:DO-41
- added J1: USB-C Receptacle, Connector:USB_C_Receptacle
- added LED1: Common Cathode RGB LED, LED:LED_RGB_TH
- added M1: Coin Vibration Motor, Connector:Connector_2pin
- added Q1, Q2, Q3, Q4: 2N2222 NPN, Package_TO_SOT_SMD:TO-92
- added R1, R15, R16, R17, R2, R3, R4, R5, R6, R7, R8: 220, Resistor_THT:R_Axial_DIN0207_L3.6mm_D1.6mm_P2.54mm_Horizontal
- added R10, R11, R12, R9: 4.7k, Resistor_THT:R_Axial_DIN0207_L3.6mm_D1.6mm_P2.54mm_Horizontal
- added R13: 10k, Resistor_THT:R_Axial_DIN0207_L3.6mm_D1.6mm_P2.54mm_Horizontal
- added R14: 12k, Resistor_THT:R_Axial_DIN0207_L3.6mm_D1.6mm_P2.54mm_Horizontal
- added R18: 1k, Resistor_THT:R_Axial_DIN0207_L3.6mm_D1.6mm_P2.54mm_Horizontal
- added R19, R20: 100k, Resistor_THT:R_Axial_DIN0207_L3.6mm_D1.6mm_P2.54mm_Horizontal
- added R_LDR: Photoresistor GL5528, Resistor_THT:R_Axial_DIN0207_L3.6mm_D1.6mm_P2.54mm_Horizontal
- added SW1, SW2: Tactile Button, Button:Switch_Tactile
- added U1: ESP32-C3 SuperMini, Connector:Header_2x13_2.54mm
- added U2: 5643A-1 4-digit 7-segment, Connector:Header_2x07_2.54mm
- added U3: TP4056 Li-Po Charger, Package_DIP:DIP-8
- added U4: MCP1700-33 3.3V LDO, Package_TO_SOT_SMD:TO-92
Other:
- title: (none) -> ESP32-C3 SuperMini Watch

Commit message: Fix KiCad 6 schematic format: flat top-level S-expressions
- Each top-level element is its own (..) group, not nested inside kicad_sch
- Format: (kicad_sch) (version 20211014) (generator eeschema) ... (matches KiCad 6 spec)
- Eeschema 10.0 loads successfully
- 39 symbols, 91 wires, 44 labels — balanced S-expression
- LDO_OUT connected to 3V3 rail, U1.VBUS connected to VBUS rail
Parts:
- removed BT1: 3.7V 150mAh Li-Po, Connector:JST_PH_2pin
- removed C1, C2: 1uF, Capacitor_THT:CP_Radial_D5.0mm_P2.50mm
- removed D1: 1N5819 Schottky (BAT→LDO), Package_TO_SOT_SMD:DO-41
- removed D2: 1N5819 Schottky (USB→LDO), Package_TO_SOT_SMD:DO-41
- removed J1: USB-C Receptacle, Connector:USB_C_Receptacle
- removed LED1: Common Cathode RGB LED, LED:LED_RGB_TH
- removed M1: Coin Vibration Motor, Connector:Connector_2pin
- removed Q1, Q2, Q3, Q4: 2N2222 NPN, Package_TO_SOT_SMD:TO-92
- removed R1, R15, R16, R17, R2, R3, R4, R5, R6, R7, R8: 220, Resistor_THT:R_Axial_DIN0207_L3.6mm_D1.6mm_P2.54mm_Horizontal
- removed R10, R11, R12, R9: 4.7k, Resistor_THT:R_Axial_DIN0207_L3.6mm_D1.6mm_P2.54mm_Horizontal
- removed R13: 10k, Resistor_THT:R_Axial_DIN0207_L3.6mm_D1.6mm_P2.54mm_Horizontal
- removed R14: 12k, Resistor_THT:R_Axial_DIN0207_L3.6mm_D1.6mm_P2.54mm_Horizontal
- removed R18: 1k, Resistor_THT:R_Axial_DIN0207_L3.6mm_D1.6mm_P2.54mm_Horizontal
- removed R19, R20: 100k, Resistor_THT:R_Axial_DIN0207_L3.6mm_D1.6mm_P2.54mm_Horizontal
- removed R_LDR: Photoresistor GL5528, Resistor_THT:R_Axial_DIN0207_L3.6mm_D1.6mm_P2.54mm_Horizontal
- removed SW1, SW2: Tactile Button, Button:Switch_Tactile
- removed U1: ESP32-C3 SuperMini, Connector:Header_2x13_2.54mm
- removed U2: 5643A-1 4-digit 7-segment, Connector:Header_2x07_2.54mm
- removed U3: TP4056 Li-Po Charger, Package_DIP:DIP-8
- removed U4: MCP1700-33 3.3V LDO, Package_TO_SOT_SMD:TO-92
Other:
- title: ESP32-C3 SuperMini Watch -> (none)

Commit message: Fix KiCad 6 schematic format: everything nested inside kicad_sch
- All top-level elements nested inside (kicad_sch ...) as KiCad 6 expects
- Format: (kicad_sch (version ...) (generator ...) ...)
- Eeschema 10.0 loads successfully
- 39 symbols, 91 wires, 44 labels — balanced S-expression
- LDO_OUT connected to 3V3 rail, U1.VBUS connected to VBUS rail
Parts:
- added BT1: 3.7V 150mAh Li-Po, Connector:JST_PH_2pin
- added C1, C2: 1uF, Capacitor_THT:CP_Radial_D5.0mm_P2.50mm
- added D1: 1N5819 Schottky (BAT→LDO), Package_TO_SOT_SMD:DO-41
- added D2: 1N5819 Schottky (USB→LDO), Package_TO_SOT_SMD:DO-41
- added J1: USB-C Receptacle, Connector:USB_C_Receptacle
- added LED1: Common Cathode RGB LED, LED:LED_RGB_TH
- added M1: Coin Vibration Motor, Connector:Connector_2pin
- added Q1, Q2, Q3, Q4: 2N2222 NPN, Package_TO_SOT_SMD:TO-92
- added R1, R15, R16, R17, R2, R3, R4, R5, R6, R7, R8: 220, Resistor_THT:R_Axial_DIN0207_L3.6mm_D1.6mm_P2.54mm_Horizontal
- added R10, R11, R12, R9: 4.7k, Resistor_THT:R_Axial_DIN0207_L3.6mm_D1.6mm_P2.54mm_Horizontal
- added R13: 10k, Resistor_THT:R_Axial_DIN0207_L3.6mm_D1.6mm_P2.54mm_Horizontal
- added R14: 12k, Resistor_THT:R_Axial_DIN0207_L3.6mm_D1.6mm_P2.54mm_Horizontal
- added R18: 1k, Resistor_THT:R_Axial_DIN0207_L3.6mm_D1.6mm_P2.54mm_Horizontal
- added R19, R20: 100k, Resistor_THT:R_Axial_DIN0207_L3.6mm_D1.6mm_P2.54mm_Horizontal
- added R_LDR: Photoresistor GL5528, Resistor_THT:R_Axial_DIN0207_L3.6mm_D1.6mm_P2.54mm_Horizontal
- added SW1, SW2: Tactile Button, Button:Switch_Tactile
- added U1: ESP32-C3 SuperMini, Connector:Header_2x13_2.54mm
- added U2: 5643A-1 4-digit 7-segment, Connector:Header_2x07_2.54mm
- added U3: TP4056 Li-Po Charger, Package_DIP:DIP-8
- added U4: MCP1700-33 3.3V LDO, Package_TO_SOT_SMD:TO-92
Other:
- title: (none) -> ESP32-C3 SuperMini Watch
